File: Keyboard.kicad_sch (KiCad schematic)
At the start: 121 parts, among them U1 Raspberry_Pi_Pico

Commit message: start updating layout
Parts:
- added D61: Diode, ScottoKeebs_Components:Diode_DO-35, symbol ScottoKeebs:Placeholder_Diode
- added S61: Keyswitch, ScottoKeebs_MX:MX_PCB_1.00u, symbol ScottoKeebs:Placeholder_Keyswitch
- S14: footprint ScottoKeebs_MX:MX_PCB_1.00u -> ScottoKeebs_MX:MX_PCB_2.00u
- S15, S28: footprint ScottoKeebs_MX:MX_PCB_1.00u -> ScottoKeebs_MX:MX_PCB_1.50u
- S29: footprint ScottoKeebs_MX:MX_PCB_1.00u -> ScottoKeebs_MX:MX_PCB_1.75u
- S41: footprint ScottoKeebs_MX:MX_PCB_1.00u -> ScottoKeebs_MX:MX_PCB_2.25u
- S42, S53: footprint ScottoKeebs_MX:MX_PCB_1.00u -> ScottoKeebs_MX:MX_PCB_2.50u
- S54, S55, S56, S58: footprint ScottoKeebs_MX:MX_PCB_1.00u -> ScottoKeebs_MX:MX_PCB_1.25u
- S57: footprint ScottoKeebs_MX:MX_PCB_1.00u -> ScottoKeebs_MX:MX_PCB_7.00u
Connections:
- net Column 1: now also S61.1
- net Row 5: now also D61.1 (K)
- new net: D61.2 (A), S61.2
Changed lines of the file:
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@@
 	)
 	(junction
+		(at 90.17 173.99)
+		(diameter 0)
+		(color 0 0 0 0)
+	)
+	(junction
 		(at 90.17 153.67)
 		(diameter 0)
@@
 	)
 	(junction
+		(at 95.25 186.69)
+		(diameter 0)
+		(color 0 0 0 0)
+	)
+	(junction
 		(at 120.65 113.03)
 		(diameter 0)
@@
 	(wire
 		(pts
+			(xy 90.17 153.67) (xy 90.17 173.99)
+		)
+		(stroke
+			(width 0)
+			(type default)
+		)
+	)
+	(wire
+		(pts
 			(xy 80.01 133.35) (xy 90.17 133.35)
 		)
@@
 	(wire
 		(pts
-			(xy 85.09 186.69) (xy 162.56 186.69)
+			(xy 85.09 186.69) (xy 95.25 186.69)
 		)
 		(stroke
@@
 	(wire
 		(pts
+			(xy 90.17 173.99) (xy 80.01 173.99)
+		)
+		(stroke
+			(width 0)
+			(type default)
+		)
+	)
+	(wire
+		(pts
 			(xy 59.69 153.67) (xy 59.69 173.99)
 		)
@@
 	(wire
 		(pts
+			(xy 95.25 186.69) (xy 162.56 186.69)
+		)
+		(stroke
+			(width 0)
+			(type default)
+		)
+	)
+	(wire
+		(pts
 			(xy 120.65 133.35) (xy 120.65 153.67)
 		)
@@
 	(wire
 		(pts
-			(xy 162.56 173.99) (xy 80.01 173.99)
+			(xy 162.56 173.99) (xy 90.17 173.99)
 		)
 		(stroke
@@
 			)
 		)
-		(property "Footprint" "ScottoKeebs_MX:MX_PCB_1.00u"
+		(property "Footprint" "ScottoKeebs_MX:MX_PCB_1.75u"
 			(at 21.59 135.89 0)
 			(effects
@@
 			)
 		)
-		(property "Footprint" "ScottoKeebs_MX:MX_PCB_1.00u"
+		(property "Footprint" "ScottoKeebs_MX:MX_PCB_7.00u"
 			(at 52.07 176.53 0)
 			(effects
@@
 	(symbol
 		(lib_id "ScottoKeebs:Placeholder_Keyswitch")
+		(at 92.71 176.53 0)
+		(unit 1)
+		(exclude_from_sim no)
+		(in_bom yes)
+		(on_board yes)
+		(dnp no)
+		(fields_autoplaced yes)
+		(property "Reference" "S61"
+			(at 92.71 168.91 0)
+			(effects
+				(font
+					(size 1.27 1.27)
+				)
+			)
+		)
+		(property "Value" "Keyswitch"
+			(at 92.71 171.45 0)
+			(effects
+				(font
+					(size 1.27 1.27)
+				)
+			)
+		)
+		(property "Footprint" "ScottoKeebs_MX:MX_PCB_1.00u"
+			(at 92.71 176.53 0)
+			(effects
+				(font
+					(size 1.27 1.27)
+				)
+				(hide yes)
+			)
+		)
+		(property "Datasheet" "~"
+			(at 92.71 176.53 0)
+			(effects
+				(font
+					(size 1.27 1.27)
+				)
+				(hide yes)
+			)
+		)
+		(property "Description" "Push button switch, normally open, two pins, 45° tilted"
+			(at 92.71 176.53 0)
+			(effects
+				(font
+					(size 1.27 1.27)
+				)
+				(hide yes)
+			)
+		)
+		(pin "2"
+		)
+		(pin "1"
+		)
+		(instances
+			(project "Keyboard"
+				(path "/df03a22e-c8dd-4eb0-8bd0-5ef69c422071"
+					(reference "S61")
+					(unit 1)
+				)
+			)
+		)
+	)
+	(symbol
+		(lib_id "ScottoKeebs:Placeholder_Keyswitch")
 		(at 133.35 96.52 0)
 		(unit 1)
@@
 			)
 		)
-		(property "Footprint" "ScottoKeebs_MX:MX_PCB_1.00u"
+		(property "Footprint" "ScottoKeebs_MX:MX_PCB_2.00u"
 			(at 153.67 96.52 0)
 			(effects
@@
 			)
 		)
-		(property "Footprint" "ScottoKeebs_MX:MX_PCB_1.00u"
+		(property "Footprint" "ScottoKeebs_MX:MX_PCB_2.50u"
 			(at 133.35 156.21 0)
 			(effects
@@
 			)
 		)
-		(property "Footprint" "ScottoKeebs_MX:MX_PCB_1.00u"
+		(property "Footprint" "ScottoKeebs_MX:MX_PCB_1.50u"
 			(at 153.67 115.57 0)
 			(effects
@@
 			)
 		)
-		(property "Footprint" "ScottoKeebs_MX:MX_PCB_1.00u"
+		(property "Footprint" "ScottoKeebs_MX:MX_PCB_1.50u"
 			(at 21.59 115.57 0)
 			(effects
@@
 	)
 	(symbol
+		(lib_id "ScottoKeebs:Placeholder_Diode")
+		(at 95.25 182.88 90)
+		(unit 1)
+		(exclude_from_sim no)
+		(in_bom yes)
+		(on_board yes)
+		(dnp no)
+		(fields_autoplaced yes)
+		(property "Reference" "D61"
+			(at 97.79 181.6099 90)
+			(effects
+				(font
+					(size 1.27 1.27)
+				)
+				(justify right)
+			)
+		)
+		(property "Value" "Diode"
+			(at 97.79 184.1499 90)
+			(effects
+				(font
+					(size 1.27 1.27)
+				)
+				(justify right)
+			)
+		)
+		(property "Footprint" "ScottoKeebs_Components:Diode_DO-35"
+			(at 95.25 182.88 0)
+			(effects
+				(font
+					(size 1.27 1.27)
+				)
+				(hide yes)
+			)
+		)
+		(property "Datasheet" ""
+			(at 95.25 182.88 0)
+			(effects
+				(font
+					(size 1.27 1.27)
+				)
+				(hide yes)
+			)
+		)
+		(property "Description" "1N4148 (DO-35) or 1N4148W (SOD-123)"
+			(at 95.25 182.88 0)
+			(effects
+				(font
+					(size 1.27 1.27)
+				)
+				(hide yes)
+			)
+		)
+		(property "Sim.Device" "D"
+			(at 95.25 182.88 0)
+			(effects
+				(font
+					(size 1.27 1.27)
+				)
+				(hide yes)
+			)
+		)
+		(property "Sim.Pins" "1=K 2=A"
+			(at 95.25 182.88 0)
+			(effects
+				(font
+					(size 1.27 1.27)
+				)
+				(hide yes)
+			)
+		)
+		(pin "1"
+		)
+		(pin "2"
+		)
+		(instances
+			(project "Keyboard"
+				(path "/df03a22e-c8dd-4eb0-8bd0-5ef69c422071"
+					(reference "D61")
+					(unit 1)
+				)
+			)
+		)
+	)
+	(symbol
 		(lib_id "ScottoKeebs:Placeholder_Keyswitch")
 		(at 123.19 135.89 0)
@@
 			)
 		)
-		(property "Footprint" "ScottoKeebs_MX:MX_PCB_1.00u"
+		(property "Footprint" "ScottoKeebs_MX:MX_PCB_1.25u"
 			(at 62.23 176.53 0)
 			(effects
@@
 			)
 		)
-		(property "Footprint" "ScottoKeebs_MX:MX_PCB_1.00u"
+		(property "Footprint" "ScottoKeebs_MX:MX_PCB_1.25u"
 			(at 31.75 176.53 0)
 			(effects
@@
 			)
 		)
-		(property "Footprint" "ScottoKeebs_MX:MX_PCB_1.00u"
+		(property "Footprint" "ScottoKeebs_MX:MX_PCB_1.25u"
 			(at 41.91 176.53 0)
 			(effects
@@
 			)
 		)
-		(property "Footprint" "ScottoKeebs_MX:MX_PCB_1.00u"
+		(property "Footprint" "ScottoKeebs_MX:MX_PCB_2.25u"
 			(at 143.51 135.89 0)
 			(effects
@@
 			)
 		)
-		(property "Footprint" "ScottoKeebs_MX:MX_PCB_1.00u"
+		(property "Footprint" "ScottoKeebs_MX:MX_PCB_1.25u"
 			(at 21.59 176.53 0)
 			(effects
@@
 			)
 		)
-		(property "Footprint" "ScottoKeebs_MX:MX_PCB_1.00u"
+		(property "Footprint" "ScottoKeebs_MX:MX_PCB_2.50u"
 			(at 21.59 156.21 0)
 			(effects
