File: Keyboard.kicad_pcb (KiCad board)
At the start: 2 copper layers, 121 parts, among them U1 Raspberry_Pi_Pico

Commit message: start updating layout
Parts:
- added D61: Diode, ScottoKeebs_Components:Diode_DO-35, F.Cu at (448.2, 50.5)
- added S61: Keyswitch, ScottoKeebs_MX:MX_PCB_1.00u, F.Cu at (395.7, 105.9)
- S14: footprint ScottoKeebs_MX:MX_PCB_1.00u -> ScottoKeebs_MX:MX_PCB_2.00u
- S15, S28: footprint ScottoKeebs_MX:MX_PCB_1.00u -> ScottoKeebs_MX:MX_PCB_1.50u
- S29: footprint ScottoKeebs_MX:MX_PCB_1.00u -> ScottoKeebs_MX:MX_PCB_1.75u
- S41: footprint ScottoKeebs_MX:MX_PCB_1.00u -> ScottoKeebs_MX:MX_PCB_2.25u
- S42, S53: footprint ScottoKeebs_MX:MX_PCB_1.00u -> ScottoKeebs_MX:MX_PCB_2.50u
- S54, S55, S56, S58: footprint ScottoKeebs_MX:MX_PCB_1.00u -> ScottoKeebs_MX:MX_PCB_1.25u
- S57: footprint ScottoKeebs_MX:MX_PCB_1.00u -> ScottoKeebs_MX:MX_PCB_7.00u
- moved U1 377.5 mm to (415.6, 93.0), turned to 0 degrees
- moved D57 337.2 mm to (448.2, 36.3)
- moved D58 337.2 mm to (448.2, 39.9)
- moved D59 337.2 mm to (448.2, 43.4)
- moved D60 337.2 mm to (448.2, 47.0)
- moved D14 337.0 mm to (415.9, 22.1)
- moved D15 337.0 mm to (415.9, 25.7)
- moved D42 337.0 mm to (437.4, 29.2)
- moved D43 337.0 mm to (437.4, 32.8)
- moved D44 337.0 mm to (437.4, 36.3)
- moved D45 337.0 mm to (437.4, 39.9)
- moved D27 336.9 mm to (426.6, 22.1)
- moved D28 336.9 mm to (426.6, 25.7)
- moved D29 336.9 mm to (426.6, 29.2)
- moved D30 336.9 mm to (426.6, 32.8)
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
Commit message: update layout and start wiring
Parts:
- D1, D10, D11, D12, D13, D14, D15, D16, D17, D18, D19, D2, D20, D21, D22, D23, D24, D25, D26, D27, D28, D29, D3, D30, D31, D32, D33, D34, D35, D36, D37, D38, D39, D4, D40, D41, D42, D43, D44, D45, D46, D47, D48, D49, D5, D50, D51, D52, D53, D54, D55, D56, D57, D58, D59, D6, D60, D61, D7, D8, D9: moved to B.Cu
- moved D54 448.1 mm to (16.9, 147.2)
- moved D55 424.2 mm to (40.7, 147.2)
- moved D42 420.4 mm to (28.8, 128.2)
- moved D29 412.8 mm to (21.6, 109.2)
- moved D56 400.4 mm to (64.5, 147.2)
- moved D25 397.7 mm to (19.3, 90.1)
- moved D1 393.6 mm to (14.5, 71.0)
- moved D43 387.2 mm to (62.1, 128.2)
- moved D30 386.4 mm to (47.8, 109.2)
- moved U1 385.6 mm to (34.8, 31.8), turned to 90 degrees
- moved D2 374.3 mm to (33.5, 71.0)
- moved D24 374.2 mm to (43.1, 90.1)
- moved D44 367.9 mm to (81.2, 128.2)
- moved D31 367.0 mm to (66.9, 109.2)
- moved D23 355.6 mm to (62.1, 90.1)
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Routing:
- net Net-(D5-A): track 0.00 -> 15.4 mm
- net Net-(D14-A): track 0.00 -> 15.1 mm
- net Net-(D8-A): track 0.00 -> 15.1 mm
- net Net-(D6-A): track 0.00 -> 15.1 mm
- net Net-(D13-A): track 0.00 -> 15.1 mm
- net Net-(D10-A): track 0.00 -> 15.1 mm
- net Net-(D2-A): track 0.00 -> 15.1 mm
- net Net-(D1-A): track 0.00 -> 15.1 mm
- net Net-(D3-A): track 0.00 -> 15.1 mm
- net Net-(D9-A): track 0.00 -> 15.1 mm
- net Net-(D11-A): track 0.00 -> 15.1 mm
- net Net-(D7-A): track 0.00 -> 15.1 mm
- net Net-(D12-A): track 0.00 -> 15.1 mm

Commit message: Continued working on wiring
Parts:
- moved D15 195.3 mm to (19.3, 90.1)
- moved D25 195.3 mm to (214.5, 90.1)
- moved D16 152.4 mm to (43.1, 90.1)
- moved D24 152.4 mm to (195.5, 90.1)
- moved D17 114.3 mm to (62.1, 90.1)
- moved D23 114.3 mm to (176.4, 90.1)
- moved D18 76.2 mm to (81.2, 90.1)
- moved D22 76.2 mm to (157.4, 90.1)
- moved D19 38.1 mm to (100.2, 90.1)
- moved D21 38.1 mm to (138.3, 90.1)
- moved D60 19.1 mm to (262.1, 147.3)
- moved D61 19.1 mm to (281.2, 147.2)
- moved S60 19.1 mm to (265.9, 137.7)
- moved S61 19.1 mm to (285.0, 137.7)
Routing:
- net Column 1: track 0.00 -> 1659.6 mm, vias 0 -> 7
- net Net-(D37-A): track 0.00 -> 15.5 mm
- net Net-(D42-A): track 0.00 -> 15.1 mm
- net Net-(D28-A): track 0.00 -> 15.1 mm
- net Net-(D27-A): track 0.00 -> 15.1 mm
- net Net-(D39-A): track 0.00 -> 15.1 mm
- net Net-(D36-A): track 0.00 -> 15.1 mm
- net Net-(D34-A): track 0.00 -> 15.1 mm
- net Net-(D30-A): track 0.00 -> 15.1 mm
- net Net-(D50-A): track 0.00 -> 15.1 mm
- net Net-(D49-A): track 0.00 -> 15.1 mm
- net Net-(D48-A): track 0.00 -> 15.1 mm
- net Net-(D47-A): track 0.00 -> 15.1 mm
- net Net-(D46-A): track 0.00 -> 15.1 mm
- net Net-(D29-A): track 0.00 -> 15.1 mm
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
Commit message: More wiring
Routing:
- net Column 1: track 1659.6 -> 3456.7 mm, vias 7 -> 27
- net Row 5: track 0.00 -> 146.7 mm
- net unconnected-(D42-K-Pad1): track 0.00 -> 4.86 mm
